File: hw/R2P_IR_module.brd (EAGLE design)
At the start: 40 x 40 mm, 32 parts, among them U1 STM32F103CX, U5 LD3985XX, X1 MICROMATCH-4

Commit message: Ongoing board layout
Parts:
- added JP3, JP4, JP5, JP6: (no value), misc:1X03
- added U$2, U$3, U$5, U$6: JST-PH3, jst:JST-PH3
Connections:
- new net +VBUS: 1.P$1, 1.P$2, 1.P$3, 2.P$1, 2.P$2, 2.P$3, JP1.1, JP2.1, R4.2, X1.1
- new net N$6: JP4.2, U$3.2
- new net N$7: JP6.2, U$6.2
- new net N$8: JP5.2, U$5.2
- net +5V: now also C7.1, JP3.1, JP4.1, JP5.1, JP6.1, R4.1, U$2.1, U$3.1, U$5.1, U$6.1, U5.1, U5.3; no longer 1.P$1, 1.P$2, 1.P$3, 2.P$1, 2.P$2, 2.P$3, JP1.1, JP2.1, R4.2, X1.1
- net GND: now also JP3.3, JP4.3, JP5.3, JP6.3, U$2.3, U$3.3, U$5.3, U$6.3
- net N$5: now also JP3.2, U$2.2; no longer C7.1, R4.1, U5.1, U5.3
Routing:
- net +VBUS: track 0.00 -> 51.4 mm
- net +5V: track 51.4 -> 86.1 mm, vias 0 -> 1
- net N$5: track 6.85 -> 3.18 mm
- net N$6: track 0.00 -> 3.18 mm
- net N$8: track 0.00 -> 3.17 mm
- net N$7: track 0.00 -> 3.17 mm
- added copper zone on layer 16, net +VBUS
- removed copper zone on layer 16, net +5V

Commit message: Board layout complete
Parts:
- added R5, R6, R7, R8: (no value), rcl:R0603
Connections:
- net +VBUS renamed +V
- removed net AM_DRDY: U1.41
- removed net AM_INT1: U1.42
- removed net AM_INT2: U1.43
- removed net GPS_RESET: U1.14
- removed net GPS_RX: U1.13
- removed net GPS_STATUS: U1.11
- removed net GPS_TX: U1.12
- removed net GYRO_CS: U1.18
- removed net GYRO_INT1: U1.21
- removed net GYRO_INT2: U1.19
- removed net MISO: U1.16
- removed net MOSI: U1.17
- removed net N$1: U$4.P$5
- removed net OSC_OUT: U1.6
- removed net SCK: U1.15
- removed net SCL: U1.45
- removed net SDA: U1.46
- new net IR1: R5.1, U1.11
- new net IR2: R6.1, U1.12
- new net IR3: R7.1, U1.19
- new net IR4: R8.1, U1.18
- net GND: now also U$4.P$5
- net N$5: now also R5.2
- net N$6: now also R6.2
- net N$7: now also R8.2
- net N$8: now also R7.2
Routing:
- net N$5: track 3.18 -> 22.0 mm
- net N$8: track 3.17 -> 13.8 mm
- net IR2: track 0.00 -> 7.92 mm
- net IR1: track 0.00 -> 7.53 mm
- net N$6: track 3.18 -> 9.28 mm
- net IR3: track 0.00 -> 6.02 mm
- net IR4: track 0.00 -> 5.37 mm
- net N$7: track 3.17 -> 6.07 mm
Changed lines of the file:
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@@
 <param name="dpGapFactor" value="2.5"/>
 <param name="checkGrid" value="0"/>
-<param name="checkAngle" value="1"/>
+<param name="checkAngle" value="0"/>
 <param name="checkFont" value="1"/>
 <param name="checkRestrict" value="0"/>
@@
 <element name="JP5" library="misc" package="1X03" value="" x="5.715" y="24.4475" rot="R180"/>
 <element name="JP6" library="misc" package="1X03" value="" x="15.24" y="24.4475" rot="R180"/>
+<element name="R5" library="rcl" package="R0603" value="" x="22.86" y="35.56" rot="R90"/>
+<element name="R6" library="rcl" package="R0603" value="" x="20.79625" y="35.56" rot="R90"/>
+<element name="R7" library="rcl" package="R0603" value="" x="15.24" y="19.84375" rot="R180"/>
+<element name="R8" library="rcl" package="R0603" value="" x="15.24" y="21.9075" rot="R180"/>
 </elements>
 <signals>
@@
 <contactref element="JP4" pad="3"/>
 <contactref element="JP3" pad="3"/>
+<contactref element="U$4" pad="P$5"/>
 </signal>
 <signal name="+3V3">
@@
 <wire x1="25.9375" y1="31.53" x2="25.9375" y2="32.195" width="0.2032" layer="1"/>
 </signal>
-<signal name="OSC_OUT">
-<contactref element="U1" pad="6"/>
-</signal>
 <signal name="NRST">
 <contactref element="U1" pad="7"/>
@@
 <wire x1="24.92375" y1="26.3525" x2="30.32125" y2="26.3525" width="0.2032" layer="16"/>
 <wire x1="30.32125" y1="26.3525" x2="32.54375" y2="28.575" width="0.2032" layer="16"/>
-</signal>
-<signal name="N$1">
-<contactref element="U$4" pad="P$5"/>
-</signal>
-<signal name="SCK">
-<contactref element="U1" pad="15"/>
-</signal>
-<signal name="MISO">
-<contactref element="U1" pad="16"/>
-</signal>
-<signal name="MOSI">
-<contactref element="U1" pad="17"/>
 </signal>
 <signal name="UART_TX">
@@
 <wire x1="28.73375" y1="8.5725" x2="29.492" y2="7.81425" width="0.2032" layer="16"/>
 </signal>
-<signal name="GYRO_CS">
-<contactref element="U1" pad="18"/>
-</signal>
-<signal name="GYRO_INT1">
-<contactref element="U1" pad="21"/>
-</signal>
-<signal name="GYRO_INT2">
-<contactref element="U1" pad="19"/>
-</signal>
 <signal name="N$4">
 <contactref element="U5" pad="4"/>
@@
 <wire x1="33.02" y1="12.8025" x2="30.99375" y2="12.8025" width="0.2032" layer="1"/>
 <wire x1="30.99375" y1="12.8025" x2="30.98625" y2="12.795" width="0.2032" layer="1"/>
-</signal>
-<signal name="SCL">
-<contactref element="U1" pad="45"/>
-</signal>
-<signal name="SDA">
-<contactref element="U1" pad="46"/>
-</signal>
-<signal name="AM_INT1">
-<contactref element="U1" pad="42"/>
-</signal>
-<signal name="AM_DRDY">
-<contactref element="U1" pad="41"/>
-</signal>
-<signal name="AM_INT2">
-<contactref element="U1" pad="43"/>
-</signal>
-<signal name="GPS_TX">
-<contactref element="U1" pad="12"/>
-</signal>
-<signal name="GPS_RX">
-<contactref element="U1" pad="13"/>
-</signal>
-<signal name="GPS_RESET">
-<contactref element="U1" pad="14"/>
-</signal>
-<signal name="GPS_STATUS">
-<contactref element="U1" pad="11"/>
 </signal>
 <signal name="BOOT0">
@@
 <wire x1="17.78" y1="24.4475" x2="17.78" y2="25.7175" width="0.6096" layer="16"/>
 </signal>
-<signal name="+VBUS">
+<signal name="+V">
 <contactref element="R4" pad="2"/>
 <polygon width="0.2032" layer="16" thermals="no">
@@
 <contactref element="JP3" pad="2"/>
 <wire x1="5.715" y1="35.08375" x2="5.715" y2="31.90875" width="0.2032" layer="16"/>
+<contactref element="R5" pad="2"/>
+<wire x1="22.86" y1="36.41" x2="22.86" y2="36.83" width="0.2032" layer="1"/>
+<wire x1="22.86" y1="36.83" x2="22.225" y2="37.465" width="0.2032" layer="1"/>
+<wire x1="22.225" y1="37.465" x2="8.09625" y2="37.465" width="0.2032" layer="1"/>
+<wire x1="8.09625" y1="37.465" x2="5.715" y2="35.08375" width="0.2032" layer="1"/>
 </signal>
 <signal name="N$6">
@@
 <contactref element="JP4" pad="2"/>
 <wire x1="15.24" y1="35.08375" x2="15.24" y2="31.90875" width="0.2032" layer="16"/>
+<contactref element="R6" pad="2"/>
+<wire x1="20.79625" y1="36.41" x2="16.56625" y2="36.41" width="0.2032" layer="1"/>
+<wire x1="16.56625" y1="36.41" x2="15.24" y2="35.08375" width="0.2032" layer="1"/>
 </signal>
 <signal name="N$7">
@@
 <contactref element="JP6" pad="2"/>
 <wire x1="15.24" y1="27.6225" x2="15.24" y2="24.4475" width="0.2032" layer="16"/>
+<contactref element="R8" pad="2"/>
+<wire x1="14.39" y1="21.9075" x2="14.39" y2="23.5975" width="0.2032" layer="1"/>
+<wire x1="14.39" y1="23.5975" x2="15.24" y2="24.4475" width="0.2032" layer="1"/>
 </signal>
 <signal name="N$8">
@@
 <contactref element="JP5" pad="2"/>
 <wire x1="5.715" y1="27.6225" x2="5.715" y2="24.4475" width="0.2032" layer="16"/>
+<contactref element="R7" pad="2"/>
+<wire x1="14.39" y1="19.84375" x2="10.31875" y2="19.84375" width="0.2032" layer="1"/>
+<wire x1="10.31875" y1="19.84375" x2="5.715" y2="24.4475" width="0.2032" layer="1"/>
+</signal>
+<signal name="IR2">
+<contactref element="R6" pad="1"/>
+<contactref element="U1" pad="12"/>
+<wire x1="22.3325" y1="27.4275" x2="22.3325" y2="29.42" width="0.2032" layer="1"/>
+<wire x1="22.3325" y1="29.42" x2="20.955" y2="30.7975" width="0.2032" layer="1"/>
+<wire x1="20.79625" y1="34.71" x2="20.79625" y2="30.95625" width="0.2032" layer="1"/>
+<wire x1="20.79625" y1="30.95625" x2="20.955" y2="30.7975" width="0.2032" layer="1"/>
+</signal>
+<signal name="IR1">
+<contactref element="R5" pad="1"/>
+<contactref element="U1" pad="11"/>
+<wire x1="22.8325" y1="27.4275" x2="22.8325" y2="29.555" width="0.2032" layer="1"/>
+<wire x1="22.8325" y1="29.555" x2="22.5425" y2="29.845" width="0.2032" layer="1"/>
+<wire x1="22.5425" y1="29.845" x2="22.5425" y2="31.115" width="0.2032" layer="1"/>
+<wire x1="22.5425" y1="31.115" x2="22.86" y2="31.4325" width="0.2032" layer="1"/>
+<wire x1="22.86" y1="31.4325" x2="22.86" y2="34.71" width="0.2032" layer="1"/>
+</signal>
+<signal name="IR3">
+<contactref element="R7" pad="1"/>
+<contactref element="U1" pad="19"/>
+<wire x1="20.8325" y1="22.9275" x2="19.91125" y2="22.9275" width="0.2032" layer="1"/>
+<wire x1="16.09" y1="19.84375" x2="16.8275" y2="19.84375" width="0.2032" layer="1"/>
+<wire x1="16.8275" y1="19.84375" x2="19.91125" y2="22.9275" width="0.2032" layer="1"/>
+</signal>
+<signal name="IR4">
+<contactref element="R8" pad="1"/>
+<contactref element="U1" pad="18"/>
+<wire x1="20.8325" y1="23.4275" x2="19.77625" y2="23.4275" width="0.2032" layer="1"/>
+<wire x1="19.77625" y1="23.4275" x2="18.25625" y2="21.9075" width="0.2032" layer="1"/>
+<wire x1="18.25625" y1="21.9075" x2="16.09" y2="21.9075" width="0.2032" layer="1"/>
 </signal>
 </signals>

Commit message: Added PMOS to shut down IR sensors
Parts:
- added R9: (no value), rcl:R0603
- added T1: (no value), zetex:SOT-23
Connections:
- new net IREN: R9.1, T1.3, U1.22
- new net VIR: JP3.1, JP4.1, JP5.1, JP6.1, T1.1, U$2.1, U$3.1, U$5.1, U$6.1
- net +5V: now also R9.2, T1.2; no longer JP3.1, JP4.1, JP5.1, JP6.1, U$2.1, U$3.1, U$5.1, U$6.1
Routing:
- net +5V: track 86.1 -> 14.0 mm, vias 1 -> 0
- net VIR: track 0.00 -> 49.7 mm
- net IREN: track 0.00 -> 15.4 mm, vias 0 -> 2
- net N$8: track 13.8 -> 15.4 mm
